File: Hardware/SIC.brd (EAGLE design)
At the start: 91.4 x 84.1 mm, 48 parts, among them IC1 MEGA8-P, IC2 7805TV, IC4 LM385-2.5, IC5 LM358N, J1 AVR_SPI_PRG_6PTH, Q1 IRF540, Q2 16MHz, X1 PTC, X2 HEATER, X3 AC

Commit message: Updated schematic
Parts:
- Q2: value 16MHz -> 8MHz
Changed lines of the file:
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@@
 <element name="R11" library="resistor" package="0207/10" value="10k" x="30.48" y="34.29" rot="R90"/>
 <element name="R12" library="resistor" package="0207/10" value="1k" x="72.39" y="26.67" rot="R90"/>
-<element name="Q2" library="special" package="QS" value="16MHz" x="41.91" y="58.42" rot="R90"/>
+<element name="Q2" library="special" package="QS" value="8MHz" x="41.91" y="58.42" rot="R90"/>
 <element name="T1" library="transistor" package="TO92-EBC" value="" x="64.77" y="33.02" rot="R90"/>
 <element name="X1" library="con-ptr500" package="AK300/2" value="PTC" x="52.07" y="29.21">
