File: Hardware/SIC.sch (EAGLE design)
At the start: 48 parts, among them IC1 MEGA8-P, IC2 7805TV, IC4 LM385-2.5, IC5 LM358N, J1 AVR_SPI_PRG_6PTH, Q1 IRF540, Q2 16MHz, X1 PTC, X2 HEATER, X3 AC

Commit message: Updated schematic
Parts:
- Q2: value 16MHz -> 8MHz
Changed lines of the file:
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@@
 <part name="R11" library="resistor" deviceset="R-EU_" device="0207/10" value="10k"/>
 <part name="R12" library="resistor" deviceset="R-EU_" device="0207/10" value="1k"/>
-<part name="Q2" library="special" deviceset="XTAL/S" device="" value="16MHz"/>
+<part name="Q2" library="special" deviceset="XTAL/S" device="" value="8MHz"/>
 <part name="U$1" library="SparkFun" deviceset="5V" device=""/>
 <part name="U$2" library="SparkFun" deviceset="5V" device=""/>
